File: Doc/RefOsc10MHz_3V0.brd (EAGLE design)
At the start: 140.8 x 317.6 mm, 70 parts, among them CON1 MCX-J-P-X-RA-SM1, CON2 TYCO-AMP_USBUSB-B_SMT, CON3 SD-73100-0105, CON4 AVR-ISP-6SMD, CON5 AVR-JTAG-10SMD, CON6 HEADER-2X3SMD, CON7 MCX-J-P-X-RA-SM1, IC11 712-RXM-GNSS-TM-B, IC3 74HCT221D, IC4 CFPT-141

Commit message: avr_DF4IAH_Bootloader - Doc - Eagle: V3.0 - REAR panel connected
Parts:
- removed R61: 51, rcl:R0805
- added CON10, CON8, CON9: MCX-J-P-X-RA-SM1, df4iah:MCX-J-P-X-RA-SM1
- added R10: 51, rcl:R0805
- added U$17, U$18, U$19, U$20, U$21, U$22, U$23, U$24, U$25, U$26, U$27, U$28, U$29, U$30, U$31, U$32: (no value), holes:2,8
- CON1: value MCX-J-P-X-RA-SM1 -> SD-73100-0105; device df4iah:MCX-J-P-X-RA-SM1 -> df4iah:MOLEX_BNC-JACK-50R_SD-73100-0105
- CON3: value SD-73100-0105 -> MCX-J-P-X-RA-SM1; device df4iah:MOLEX_BNC-JACK-50R_SD-73100-0105 -> df4iah:MCX-J-P-X-RA-SM1
- moved CON3 648.0 mm to (-143.5, -577.9), turned to 0 degrees
- moved CON1 233.9 mm to (16.3, -303.6), turned to 180 degrees
Connections:
- removed net C_10MHZ: R61.1
- removed net N$42: CON3.1, R61.2
- new net REFC_10MHZ: CON1.1
- new net SIG_CH0_I: CON3.1
- new net SIG_CH0_Q: CON8.1
- new net SIG_CH1_I: CON9.1
- new net SIG_CH1_Q: CON10.1
- net GND: now also CON1.2, CON1.3, CON10.2, CON10.3, CON10.4, CON10.5, CON3.4, CON3.5, CON7.2, CON7.3, CON7.4, CON7.5, CON8.2, CON8.3, CON8.4, CON8.5, CON9.2, CON9.3, CON9.4, CON9.5
- net GPS_HF: now also CON7.1
Routing:
- net C_10MHZ: track 17.5 -> 0.00 mm, vias 1 -> 0
- net N$42: track 10.7 -> 0.00 mm, vias 1 -> 0
- net GND3: track 0.00 -> 1.30 mm, vias 0 -> 8
- net GND2: track 0.00 -> 1.30 mm, vias 0 -> 8
- added copper zone on layer 16, net GND2
- added copper zone on layer 16, net GND3
Other:
- board size 140.8 x 317.6 mm -> 214.5 x 647.9 mm

Commit message: avr_DF4IAH_Bootloader - Doc - Eagle: V3.0 - FPGA and MMU, first attempt, added
Parts:
- added IC1: XMEGA128A1, atmel:TQFP100
- added R1: 200, rcl:R0805
- added U1: 6SLX4TQG144, xilinx_devices_V6:TQ144
Connections:
- new net AVCC1: IC1.94
- new net GND1: IC1.13
- new net GND2: IC1.23
- new net GND3: IC1.33
- new net GND4: IC1.43
- new net GND5: IC1.53
- new net GND6: IC1.63
- new net GND7: IC1.73
- new net GND8: IC1.84
- new net GND9: IC1.93
- new net VCC1: IC1.24
- new net VCC2: IC1.34
- new net VCC3: IC1.44
- new net VCC4: IC1.54
- new net VCC5: IC1.64
- new net VCC6: IC1.74
- new net VCC7: IC1.83
- net AVCC: now also IC1.4
- net GND: now also IC1.3, U1.P108, U1.P113, U1.P13, U1.P130, U1.P136, U1.P25, U1.P3, U1.P49, U1.P54, U1.P68, U1.P77, U1.P91, U1.P96
- net VCC: now also IC1.14
Changed lines of the file:
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@@
 <element name="CON10" library="df4iah" package="MCX-J-P-X-RA-SM1" value="MCX-J-P-X-RA-SM1" x="-170.18" y="-577.85"/>
 <element name="R10" library="rcl" package="R0805" value="51" x="-171.45" y="-613.41"/>
+<element name="U1" library="xilinx_devices_V6" package="TQ144" value="6SLX4TQG144" x="-161.29" y="-628.65"/>
+<element name="R1" library="rcl" package="R0805" value="200" x="-171.45" y="-643.89"/>
+<element name="IC1" library="atmel" package="TQFP100" value="XMEGA128A1" x="-182.88" y="-637.54">
+<attribute name="OC_NEWARK" value="unknown" x="-182.88" y="-637.54" size="1.778" layer="27" display="off"/>
+<attribute name="MPN" value="" x="-182.88" y="-637.54" size="1.778" layer="27" display="off"/>
+<attribute name="MF" value="" x="-182.88" y="-637.54" size="1.778" layer="27" display="off"/>
+<attribute name="OC_FARNELL" value="unknown" x="-182.88" y="-637.54" size="1.778" layer="27" display="off"/>
+</element>
 </elements>
 <signals>
@@
 <contactref element="CON10" pad="4"/>
 <contactref element="CON10" pad="5"/>
+<contactref element="U1" pad="P3"/>
+<contactref element="U1" pad="P13"/>
+<contactref element="U1" pad="P25"/>
+<contactref element="U1" pad="P49"/>
+<contactref element="U1" pad="P54"/>
+<contactref element="U1" pad="P68"/>
+<contactref element="U1" pad="P77"/>
+<contactref element="U1" pad="P91"/>
+<contactref element="U1" pad="P96"/>
+<contactref element="U1" pad="P108"/>
+<contactref element="U1" pad="P113"/>
+<contactref element="U1" pad="P130"/>
+<contactref element="U1" pad="P136"/>
+<contactref element="IC1" pad="3"/>
 <wire x1="-172.72" y1="-575.31" x2="-172.72" y2="-580.39" width="0" layer="19" extent="1-1"/>
 <wire x1="-167.64" y1="-580.39" x2="-172.72" y2="-580.39" width="0" layer="19" extent="1-1"/>
@@
 <wire x1="-140.97" y1="-580.39" x2="-146.05" y2="-580.39" width="0" layer="19" extent="1-1"/>
 <wire x1="-140.97" y1="-575.31" x2="-146.05" y2="-575.31" width="0" layer="19" extent="1-1"/>
+<wire x1="-163.04" y1="-617.55" x2="-163.83" y2="-580.39" width="0" layer="19" extent="1-1"/>
+<wire x1="-166.04" y1="-617.55" x2="-163.04" y2="-617.55" width="0" layer="19" extent="1-1"/>
+<wire x1="-172.39" y1="-620.9" x2="-166.04" y2="-617.55" width="0" layer="19" extent="1-1"/>
+<wire x1="-172.39" y1="-625.9" x2="-172.39" y2="-620.9" width="0" layer="19" extent="1-1"/>
+<wire x1="-172.39" y1="-631.9" x2="-172.39" y2="-625.9" width="0" layer="19" extent="1-1"/>
+<wire x1="-154.54" y1="-617.55" x2="-163.04" y2="-617.55" width="0" layer="19" extent="1-1"/>
+<wire x1="-150.19" y1="-619.9" x2="-154.54" y2="-617.55" width="0" layer="19" extent="1-1"/>
+<wire x1="-150.19" y1="-625.9" x2="-150.19" y2="-619.9" width="0" layer="19" extent="1-1"/>
+<wire x1="-150.19" y1="-628.4" x2="-150.19" y2="-625.9" width="0" layer="19" extent="1-1"/>
+<wire x1="-150.19" y1="-635.4" x2="-150.19" y2="-628.4" width="0" layer="19" extent="1-1"/>
+<wire x1="-154.54" y1="-639.75" x2="-150.19" y2="-635.4" width="0" layer="19" extent="1-1"/>
+<wire x1="-161.54" y1="-639.75" x2="-154.54" y2="-639.75" width="0" layer="19" extent="1-1"/>
+<wire x1="-164.04" y1="-639.75" x2="-161.54" y2="-639.75" width="0" layer="19" extent="1-1"/>
+<wire x1="-190.88" y1="-632.54" x2="-172.39" y2="-631.9" width="0" layer="19" extent="1-1"/>
 <wire x1="11.74" y1="-307.38" x2="-140.97" y2="-575.31" width="0" layer="19" extent="1-1"/>
 <wire x1="11.74" y1="-299.78" x2="11.74" y2="-307.38" width="0" layer="19" extent="1-1"/>
@@
 <via x="20.955" y="5.08" extent="1-16" drill="0.35"/>
 <wire x1="16.8275" y1="15.25" x2="14.125" y2="15.25" width="0.508" layer="1"/>
+<contactref element="IC1" pad="14"/>
 <wire x1="49.53" y1="30.48" x2="49.8475" y2="30.7975" width="0" layer="19" extent="1-1"/>
 <wire x1="24.13" y1="16.8275" x2="24.4475" y2="16.8275" width="0" layer="19" extent="1-1"/>
@@
 <wire x1="19.3675" y1="17.4625" x2="19.3675" y2="17.78" width="0" layer="19" extent="16-16"/>
 <wire x1="20.32" y1="50.4825" x2="20.0025" y2="46.6725" width="0" layer="19" extent="16-16"/>
+<wire x1="-190.88" y1="-638.04" x2="23.1775" y2="2.8575" width="0" layer="19" extent="1-1"/>
 </signal>
 <signal name="N_ADC_PULL">
@@
 <wire x1="21.2725" y1="64.77" x2="21" y2="64.77" width="0.3" layer="16"/>
 <wire x1="24.13" y1="61.9125" x2="24.13" y2="55.88" width="0.3" layer="16"/>
+<contactref element="IC1" pad="4"/>
+<wire x1="-190.88" y1="-633.04" x2="24.13" y2="55.88" width="0" layer="19" extent="1-16"/>
 </signal>
 <signal name="ISP_SCK">
@@
 <wire x1="29.473853125" y1="-193.909359375" x2="29.445821875" y2="-193.9082875" width="0.762" layer="1"/>
 <wire x1="29.473853125" y1="-193.909359375" x2="29.40475625" y2="-193.83519375" width="0.762" layer="1"/>
+<contactref element="IC1" pad="13"/>
 <wire x1="29.428378125" y1="-194.352440625" x2="23.662771875" y2="-199.733378125" width="0" layer="19" extent="1-1"/>
 <wire x1="32.230040625" y1="-188.2886625" x2="29.448715625" y2="-193.83460625" width="0" layer="19" extent="1-1"/>
@@
 <wire x1="46.200040625" y1="-105.7386625" x2="43.418715625" y2="-111.28460625" width="0" layer="19" extent="1-1"/>
 <wire x1="26.163896875" y1="-105.008475" x2="37.632771875" y2="-117.183378125" width="0" layer="19" extent="1-1"/>
+<wire x1="-190.88" y1="-637.54" x2="23.662771875" y2="-199.733378125" width="0" layer="19" extent="1-1"/>
 </signal>
 <signal name="GND2" class="3">
@@
 <wire x1="-7.356146875" y1="-359.009359375" x2="-7.384178125" y2="-359.0082875" width="0.762" layer="1"/>
 <wire x1="-7.356146875" y1="-359.009359375" x2="-7.42524375" y2="-358.93519375" width="0.762" layer="1"/>
+<contactref element="IC1" pad="23"/>
 <wire x1="-7.401621875" y1="-359.452440625" x2="-13.167228125" y2="-364.833378125" width="0" layer="19" extent="1-1"/>
 <wire x1="-4.599959375" y1="-353.3886625" x2="-7.381284375" y2="-358.93460625" width="0" layer="19" extent="1-1"/>
@@
 <wire x1="9.370040625" y1="-270.8386625" x2="6.588715625" y2="-276.38460625" width="0" layer="19" extent="1-1"/>
 <wire x1="-10.666103125" y1="-270.108475" x2="0.802771875" y2="-282.283378125" width="0" layer="19" extent="1-1"/>
+<wire x1="-190.88" y1="-642.54" x2="-13.167228125" y2="-364.833378125" width="0" layer="19" extent="1-1"/>
 </signal>
 <signal name="GND3" class="3">
@@
 <wire x1="-44.186146875" y1="-524.109359375" x2="-44.214178125" y2="-524.1082875" width="0.762" layer="1"/>
 <wire x1="-44.186146875" y1="-524.109359375" x2="-44.25524375" y2="-524.03519375" width="0.762" layer="1"/>
+<contactref element="IC1" pad="33"/>
 <wire x1="-30.261621875" y1="-442.002440625" x2="-36.027228125" y2="-447.383378125" width="0" layer="19" extent="1-1"/>
 <wire x1="-27.459959375" y1="-435.9386625" x2="-30.241284375" y2="-441.48460625" width="0" layer="19" extent="1-1"/>
@@
 <wire x1="-49.997228125" y1="-529.933378125" x2="-44.231621875" y2="-524.552440625" width="0" layer="19" extent="1-1"/>
 <wire x1="-61.466103125" y1="-517.758475" x2="-49.997228125" y2="-529.933378125" width="0" layer="19" extent="1-1"/>
+<wire x1="-185.38" y1="-645.54" x2="-61.466103125" y2="-517.758475" width="0" layer="19" extent="1-1"/>
 </signal>
 <signal name="REFC_10MHZ">
@@
 <contactref element="CON10" pad="1"/>
 </signal>
+<signal name="AVCC1">
+<contactref element="IC1" pad="94"/>
+</signal>
+<signal name="GND9">
+<contactref element="IC1" pad="93"/>
+</signal>
+<signal name="VCC1">
+<contactref element="IC1" pad="24"/>
+</signal>
+<signal name="GND4">
+<contactref element="IC1" pad="43"/>
+</signal>
+<signal name="GND5">
+<contactref element="IC1" pad="53"/>
+</signal>
+<signal name="GND6">
+<contactref element="IC1" pad="63"/>
+</signal>
+<signal name="GND7">
+<contactref element="IC1" pad="73"/>
+</signal>
+<signal name="VCC2">
+<contactref element="IC1" pad="34"/>
+</signal>
+<signal name="VCC3">
+<contactref element="IC1" pad="44"/>
+</signal>
+<signal name="VCC4">
+<contactref element="IC1" pad="54"/>
+</signal>
+<signal name="VCC5">
+<contactref element="IC1" pad="64"/>
+</signal>
+<signal name="VCC6">
+<contactref element="IC1" pad="74"/>
+</signal>
+<signal name="VCC7">
+<contactref element="IC1" pad="83"/>
+</signal>
+<signal name="GND8">
+<contactref element="IC1" pad="84"/>
+</signal>
 </signals>

Commit message: avr_DF4IAH_Bootloader - Doc - Eagle: V3.0 - MMU (AVR ATmega) moved into FPGA using a free MMU core from opencores.org.
Parts:
- removed IC1: XMEGA128A1, atmel:TQFP100
- removed R1: 200, rcl:R0805
Connections:
- removed net AVCC1: IC1.94
- removed net GND1: IC1.13
- removed net GND2: IC1.23
- removed net GND3: IC1.33
- removed net GND4: IC1.43
- removed net GND5: IC1.53
- removed net GND6: IC1.63
- removed net GND7: IC1.73
- removed net GND8: IC1.84
- removed net GND9: IC1.93
- removed net VCC1: IC1.24
- removed net VCC2: IC1.34
- removed net VCC3: IC1.44
- removed net VCC4: IC1.54
- removed net VCC5: IC1.64
- removed net VCC6: IC1.74
- removed net VCC7: IC1.83
- net AVCC: no longer IC1.4
- net GND: no longer IC1.3
- net VCC: no longer IC1.14
Changed lines of the file:
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@@
 <?xml version="1.0" encoding="utf-8"?>
 <!DOCTYPE eagle SYSTEM "eagle.dtd">
-<eagle version="6.5.0">
+<eagle version="7.2.0">
 <drawing>
 <settings>
@@
 <pass name="Default">
 <param name="RoutingGrid" value="6.25mil"/>
+<param name="AutoGrid" value="1"/>
+<param name="Efforts" value="0"/>
+<param name="TopRouterVariant" value="1"/>
 <param name="tpViaShape" value="round"/>
 <param name="PrefDir.1" value="|"/>
@@
 <element name="R10" library="rcl" package="R0805" value="51" x="-171.45" y="-613.41"/>
 <element name="U1" library="xilinx_devices_V6" package="TQ144" value="6SLX4TQG144" x="-161.29" y="-628.65"/>
-<element name="R1" library="rcl" package="R0805" value="200" x="-171.45" y="-643.89"/>
-<element name="IC1" library="atmel" package="TQFP100" value="XMEGA128A1" x="-182.88" y="-637.54">
-<attribute name="OC_NEWARK" value="unknown" x="-182.88" y="-637.54" size="1.778" layer="27" display="off"/>
-<attribute name="MPN" value="" x="-182.88" y="-637.54" size="1.778" layer="27" display="off"/>
-<attribute name="MF" value="" x="-182.88" y="-637.54" size="1.778" layer="27" display="off"/>
-<attribute name="OC_FARNELL" value="unknown" x="-182.88" y="-637.54" size="1.778" layer="27" display="off"/>
-</element>
 </elements>
 <signals>
@@
 <contactref element="U1" pad="P130"/>
 <contactref element="U1" pad="P136"/>
-<contactref element="IC1" pad="3"/>
 <wire x1="-172.72" y1="-575.31" x2="-172.72" y2="-580.39" width="0" layer="19" extent="1-1"/>
 <wire x1="-167.64" y1="-580.39" x2="-172.72" y2="-580.39" width="0" layer="19" extent="1-1"/>
@@
 <wire x1="-161.54" y1="-639.75" x2="-154.54" y2="-639.75" width="0" layer="19" extent="1-1"/>
 <wire x1="-164.04" y1="-639.75" x2="-161.54" y2="-639.75" width="0" layer="19" extent="1-1"/>
-<wire x1="-190.88" y1="-632.54" x2="-172.39" y2="-631.9" width="0" layer="19" extent="1-1"/>
 <wire x1="11.74" y1="-307.38" x2="-140.97" y2="-575.31" width="0" layer="19" extent="1-1"/>
 <wire x1="11.74" y1="-299.78" x2="11.74" y2="-307.38" width="0" layer="19" extent="1-1"/>
@@
 <via x="20.955" y="5.08" extent="1-16" drill="0.35"/>
 <wire x1="16.8275" y1="15.25" x2="14.125" y2="15.25" width="0.508" layer="1"/>
-<contactref element="IC1" pad="14"/>
 <wire x1="49.53" y1="30.48" x2="49.8475" y2="30.7975" width="0" layer="19" extent="1-1"/>
 <wire x1="24.13" y1="16.8275" x2="24.4475" y2="16.8275" width="0" layer="19" extent="1-1"/>
@@
 <wire x1="19.3675" y1="17.4625" x2="19.3675" y2="17.78" width="0" layer="19" extent="16-16"/>
 <wire x1="20.32" y1="50.4825" x2="20.0025" y2="46.6725" width="0" layer="19" extent="16-16"/>
-<wire x1="-190.88" y1="-638.04" x2="23.1775" y2="2.8575" width="0" layer="19" extent="1-1"/>
 </signal>
 <signal name="N_ADC_PULL">
@@
 <wire x1="21.2725" y1="64.77" x2="21" y2="64.77" width="0.3" layer="16"/>
 <wire x1="24.13" y1="61.9125" x2="24.13" y2="55.88" width="0.3" layer="16"/>
-<contactref element="IC1" pad="4"/>
-<wire x1="-190.88" y1="-633.04" x2="24.13" y2="55.88" width="0" layer="19" extent="1-16"/>
 </signal>
 <signal name="ISP_SCK">
@@
 <wire x1="29.473853125" y1="-193.909359375" x2="29.445821875" y2="-193.9082875" width="0.762" layer="1"/>
 <wire x1="29.473853125" y1="-193.909359375" x2="29.40475625" y2="-193.83519375" width="0.762" layer="1"/>
-<contactref element="IC1" pad="13"/>
 <wire x1="29.428378125" y1="-194.352440625" x2="23.662771875" y2="-199.733378125" width="0" layer="19" extent="1-1"/>
 <wire x1="32.230040625" y1="-188.2886625" x2="29.448715625" y2="-193.83460625" width="0" layer="19" extent="1-1"/>
@@
 <wire x1="46.200040625" y1="-105.7386625" x2="43.418715625" y2="-111.28460625" width="0" layer="19" extent="1-1"/>
 <wire x1="26.163896875" y1="-105.008475" x2="37.632771875" y2="-117.183378125" width="0" layer="19" extent="1-1"/>
-<wire x1="-190.88" y1="-637.54" x2="23.662771875" y2="-199.733378125" width="0" layer="19" extent="1-1"/>
 </signal>
 <signal name="GND2" class="3">
@@
 <wire x1="-7.356146875" y1="-359.009359375" x2="-7.384178125" y2="-359.0082875" width="0.762" layer="1"/>
 <wire x1="-7.356146875" y1="-359.009359375" x2="-7.42524375" y2="-358.93519375" width="0.762" layer="1"/>
-<contactref element="IC1" pad="23"/>
 <wire x1="-7.401621875" y1="-359.452440625" x2="-13.167228125" y2="-364.833378125" width="0" layer="19" extent="1-1"/>
 <wire x1="-4.599959375" y1="-353.3886625" x2="-7.381284375" y2="-358.93460625" width="0" layer="19" extent="1-1"/>
@@
 <wire x1="9.370040625" y1="-270.8386625" x2="6.588715625" y2="-276.38460625" width="0" layer="19" extent="1-1"/>
 <wire x1="-10.666103125" y1="-270.108475" x2="0.802771875" y2="-282.283378125" width="0" layer="19" extent="1-1"/>
-<wire x1="-190.88" y1="-642.54" x2="-13.167228125" y2="-364.833378125" width="0" layer="19" extent="1-1"/>
 </signal>
 <signal name="GND3" class="3">
@@
 <wire x1="-44.186146875" y1="-524.109359375" x2="-44.214178125" y2="-524.1082875" width="0.762" layer="1"/>
 <wire x1="-44.186146875" y1="-524.109359375" x2="-44.25524375" y2="-524.03519375" width="0.762" layer="1"/>
-<contactref element="IC1" pad="33"/>
 <wire x1="-30.261621875" y1="-442.002440625" x2="-36.027228125" y2="-447.383378125" width="0" layer="19" extent="1-1"/>
 <wire x1="-27.459959375" y1="-435.9386625" x2="-30.241284375" y2="-441.48460625" width="0" layer="19" extent="1-1"/>
@@
 <wire x1="-49.997228125" y1="-529.933378125" x2="-44.231621875" y2="-524.552440625" width="0" layer="19" extent="1-1"/>
 <wire x1="-61.466103125" y1="-517.758475" x2="-49.997228125" y2="-529.933378125" width="0" layer="19" extent="1-1"/>
-<wire x1="-185.38" y1="-645.54" x2="-61.466103125" y2="-517.758475" width="0" layer="19" extent="1-1"/>
 </signal>
 <signal name="REFC_10MHZ">
@@
 <contactref element="CON10" pad="1"/>
 </signal>
-<signal name="AVCC1">
-<contactref element="IC1" pad="94"/>
-</signal>
-<signal name="GND9">
-<contactref element="IC1" pad="93"/>
-</signal>
-<signal name="VCC1">
-<contactref element="IC1" pad="24"/>
-</signal>
-<signal name="GND4">
-<contactref element="IC1" pad="43"/>
-</signal>
-<signal name="GND5">
-<contactref element="IC1" pad="53"/>
-</signal>
-<signal name="GND6">
-<contactref element="IC1" pad="63"/>
-</signal>
-<signal name="GND7">
-<contactref element="IC1" pad="73"/>
-</signal>
-<signal name="VCC2">
-<contactref element="IC1" pad="34"/>
-</signal>
-<signal name="VCC3">
-<contactref element="IC1" pad="44"/>
-</signal>
-<signal name="VCC4">
-<contactref element="IC1" pad="54"/>
-</signal>
-<signal name="VCC5">
-<contactref element="IC1" pad="64"/>
-</signal>
-<signal name="VCC6">
-<contactref element="IC1" pad="74"/>
-</signal>
-<signal name="VCC7">
-<contactref element="IC1" pad="83"/>
-</signal>
-<signal name="GND8">
-<contactref element="IC1" pad="84"/>
-</signal>
 </signals>

Commit message: avr_DF4IAH_Bootloader - Doc - Eagle: V3.0 - xilinx_devices_V6.lbr containing XC7-Artix added (2)
Parts:
- removed U1: 6SLX4TQG144, xilinx_devices_V6:TQ144
Connections:
- net GND: no longer U1.P108, U1.P113, U1.P13, U1.P130, U1.P136, U1.P25, U1.P3, U1.P49, U1.P54, U1.P68, U1.P77, U1.P91, U1.P96
Changed lines of the file:
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@@
 <element name="CON10" library="df4iah" package="MCX-J-P-X-RA-SM1" value="MCX-J-P-X-RA-SM1" x="-170.18" y="-577.85"/>
 <element name="R10" library="rcl" package="R0805" value="51" x="-171.45" y="-613.41"/>
-<element name="U1" library="xilinx_devices_V6" package="TQ144" value="6SLX4TQG144" x="-161.29" y="-628.65"/>
 </elements>
 <signals>
@@
 <contactref element="CON10" pad="4"/>
 <contactref element="CON10" pad="5"/>
-<contactref element="U1" pad="P3"/>
-<contactref element="U1" pad="P13"/>
-<contactref element="U1" pad="P25"/>
-<contactref element="U1" pad="P49"/>
-<contactref element="U1" pad="P54"/>
-<contactref element="U1" pad="P68"/>
-<contactref element="U1" pad="P77"/>
-<contactref element="U1" pad="P91"/>
-<contactref element="U1" pad="P96"/>
-<contactref element="U1" pad="P108"/>
-<contactref element="U1" pad="P113"/>
-<contactref element="U1" pad="P130"/>
-<contactref element="U1" pad="P136"/>
 <wire x1="-172.72" y1="-575.31" x2="-172.72" y2="-580.39" width="0" layer="19" extent="1-1"/>
 <wire x1="-167.64" y1="-580.39" x2="-172.72" y2="-580.39" width="0" layer="19" extent="1-1"/>
@@
 <wire x1="-140.97" y1="-580.39" x2="-146.05" y2="-580.39" width="0" layer="19" extent="1-1"/>
 <wire x1="-140.97" y1="-575.31" x2="-146.05" y2="-575.31" width="0" layer="19" extent="1-1"/>
-<wire x1="-163.04" y1="-617.55" x2="-163.83" y2="-580.39" width="0" layer="19" extent="1-1"/>
-<wire x1="-166.04" y1="-617.55" x2="-163.04" y2="-617.55" width="0" layer="19" extent="1-1"/>
-<wire x1="-172.39" y1="-620.9" x2="-166.04" y2="-617.55" width="0" layer="19" extent="1-1"/>
-<wire x1="-172.39" y1="-625.9" x2="-172.39" y2="-620.9" width="0" layer="19" extent="1-1"/>
-<wire x1="-172.39" y1="-631.9" x2="-172.39" y2="-625.9" width="0" layer="19" extent="1-1"/>
-<wire x1="-154.54" y1="-617.55" x2="-163.04" y2="-617.55" width="0" layer="19" extent="1-1"/>
-<wire x1="-150.19" y1="-619.9" x2="-154.54" y2="-617.55" width="0" layer="19" extent="1-1"/>
-<wire x1="-150.19" y1="-625.9" x2="-150.19" y2="-619.9" width="0" layer="19" extent="1-1"/>
-<wire x1="-150.19" y1="-628.4" x2="-150.19" y2="-625.9" width="0" layer="19" extent="1-1"/>
-<wire x1="-150.19" y1="-635.4" x2="-150.19" y2="-628.4" width="0" layer="19" extent="1-1"/>
-<wire x1="-154.54" y1="-639.75" x2="-150.19" y2="-635.4" width="0" layer="19" extent="1-1"/>
-<wire x1="-161.54" y1="-639.75" x2="-154.54" y2="-639.75" width="0" layer="19" extent="1-1"/>
-<wire x1="-164.04" y1="-639.75" x2="-161.54" y2="-639.75" width="0" layer="19" extent="1-1"/>
 <wire x1="11.74" y1="-307.38" x2="-140.97" y2="-575.31" width="0" layer="19" extent="1-1"/>
 <wire x1="11.74" y1="-299.78" x2="11.74" y2="-307.38" width="0" layer="19" extent="1-1"/>
