File: Doc/V3.x/RefOsc10MHz_3V0.brd (EAGLE design)
At the start: 214.5 x 647.9 mm, 89 parts, among them CON1 SD-73100-0105, CON10 MCX-J-P-X-RA-SM1, CON2 TYCO-AMP_USBUSB-B_SMT, CON3 MCX-J-P-X-RA-SM1, CON4 AVR-ISP-6SMD, CON5 AVR-JTAG-10SMD, CON6 HEADER-2X3SMD, CON7 MCX-J-P-X-RA-SM1, CON8 MCX-J-P-X-RA-SM1, CON9 MCX-J-P-X-RA-SM1, IC11 712-RXM-GNSS-TM-B, IC3 74HCT221D, IC4 CFPT-141

Commit message: avr_DF4IAH_Bootloader - Doc - Eagle: V3.0 - update of current dev. state
Parts:
- removed C111: 100n, df4iah:C0805
- removed C221, C31, C4: 100n, rcl:C0805
- removed C3: 47uF, rcl:PANASONIC_C
- removed C32: 100p, rcl:C0805
- removed C51, C911, C921, C922, C931, C951: 10n, rcl:C0805
- removed C71: 10p, rcl:C0805
- removed C72: 33p, rcl:C0805
- removed C81: 0.22F, rcl:PANASONIC_C
- removed CON1: SD-73100-0105, df4iah:MOLEX_BNC-JACK-50R_SD-73100-0105
- removed CON10, CON3, CON7, CON8, CON9: MCX-J-P-X-RA-SM1, df4iah:MCX-J-P-X-RA-SM1
- removed CON2: TYCO-AMP_USBUSB-B_SMT, df4iah:TYCO-AMP_USB-B_SMT
- removed CON4: AVR-ISP-6SMD, atmel-1:2X3SMD
- removed CON5: AVR-JTAG-10SMD, df4iah:2X5SMD
- removed CON6: HEADER-2X3SMD, df4iah:2X03SMD
- removed D202: BZX84-C2V7, diode:TO236
- removed D221: BZX84-C3V0, diode:TO236
- removed D3, D4: BZX84-C3V6, diode:TO236
- removed D82: CRS08, diode:SOT23
- removed IC11: 712-RXM-GNSS-TM-B, df4iah:712-RXM-GNSS-TM-B
- removed IC3: 74HCT221D, 74xx-eu:SO16
- removed IC4: CFPT-141, df4iah:CFPT-141
- removed JP1, JP2, JP3: (no value), jumper:SJW
- removed L31: 10uH, rcl:L1812
- removed LFP111: WE-CBF_300R, df4iah:L3216C
- removed R21, R22, R23, R25: 2.7k, rcl:R0805
- removed R221: 56, rcl:R0805
- removed R41: 12k, rcl:R0805
- removed R5, R6: 68, rcl:R0805
- removed R51, R52, R81: 1k, rcl:R0805
- removed R7, R71: 1.5k, rcl:R0805
- removed R8: 1M, rcl:R0805
- removed RPOLY2: 1206L012WR_0.1A, rcl:M1206
- removed RPOLY3: 1206L025YR_0.5A, rcl:M1206
- removed SJ21, SJ22: (no value), jumper:SJ
- removed U$1, U$10, U$11, U$12, U$13, U$14, U$15, U$16, U$17, U$18, U$19, U$2, U$20, U$21, U$22, U$23, U$24, U$25, U$26, U$27, U$28, U$29, U$3, U$30, U$31, U$32, U$4, U$5, U$6, U$7, U$8, U$9: (no value), holes:2,8
- added C031, C142: 100n, rcl:C0805
- added C041, C1011, C1021: 47uF, rcl:C0805
- added C051, C1001: 100uF, rcl:C1206
- added C052, C053, C062, C063, C071, C082, C083, C091, C1002, C1003, C1022, C1023: 4.7uF, rcl:C0402
- added C054, C055, C056, C057, C064, C065, C066, C067, C072, C073, C084, C085, C086, C087, C092, C1004, C1005, C1006, C1012, C1024, C1025, C1026: 0.47uF, rcl:C0402
- added C141: 47uF, rcl:PANASONIC_C
- added C151: 0.22F, rcl:PANASONIC_C
- added C152: 100n, df4iah:C0805
- added CON141: TYCO-AMP_USBUSB-B_SMT, df4iah:TYCO-AMP_USB-B_SMT
- added CON151: HEADER-2X5SMD, df4iah_connector:2X5SMD
- added CON181, CON183, CON184, CON185, CON186: MCX-J-P-X-RA-SM1, df4iah:MCX-J-P-X-RA-SM1
- added CON182: SD-73100-0105, df4iah:MOLEX_BNC-JACK-50R_SD-73100-0105
- added CON191: HEADER-2X3SMD, df4iah:2X03SMD
- added CON192: AVR-JTAG-10SMD, df4iah:2X5SMD
- added D031: BZX84-C3V0, diode:TO236
- added D141, D142: BZX84-C3V6, diode:TO236
- added D151: CRS08, diode:SOT23
- added D191: BZX84-C2V7, diode:TO236
- added H191, H192, H193, H194: MOUNT-PAD-ROUND2.8, holes:2,8-PAD
- added L191: 10uH, rcl:L1812
- added R021: 0, rcl:R0805
- added R031: 56, rcl:R0805
- added R041, R042, R051, R061, R071, R081, R091, R101, R102, R103, R104, R105: 0, rcl:R0402
- added R141, R142: 68, rcl:R0805
- added R143: 1M, rcl:R0805
- added R144: 1.5k, rcl:R0805
- added R151, R152: 10k, rcl:R0805
- added RP141: 1206L025YR_0.5A, rcl:M1206
- added RP151: 1206L012WR_0.1A, rcl:M1206
- added U031: CFPT-141, df4iah:CFPT-141
- added U1: XC7A35TFTG256, df4iah_fpga:FTG256_0MM4
- added U151: GLOBALTOP-FIREFLY1-GMM-G3, df4iah_gps:GLOBALTOP-FIREFLY1-GMM-G3
- moved R10 712.9 mm to (14.0, 74.9)
Connections:
- removed net +3V0: C221.1, D221.C, IC4.4, R221.2
- removed net +3V3: C921.1, C922.1, CON6.5, D202.C, D82.1, R221.1, RPOLY2.2, SJ22.2
- removed net 14: IC11.14, LFP111.1
- removed net ADC_PHASE: R52.2
- removed net ADC_PHASE_PULLHOLD: C51.1, R51.2
- removed net AREF: C32.1
- removed net AVCC: C31.2, L31.1
- removed net CPLD_GPS_NMEA_TX: R25.2
- removed net GND_SJ1: SJ21.2
- removed net GPS_HF: CON7.1, IC11.11, LFP111.2
- removed net INT1: JP3.2
- removed net ISP_MISO: CON4.1, R22.1
- removed net ISP_MOSI: CON4.4
- removed net ISP_SCK: CON4.3, R23.2
- removed net ISP_VTARGET: CON4.2, JP2.1
- removed net JTAG_SRST: CON4.5, CON5.6, JP1.2, R21.2
- removed net JTAG_TCK: CON5.1
- removed net JTAG_TDI: CON5.9
- removed net JTAG_TDO: CON5.3
- removed net JTAG_TMS: CON5.5
- removed net JTAG_VREF: CON5.4, R81.1
- removed net MISO: R22.2
- removed net N$1: CON6.2
- removed net N$3: CON6.4
- removed net N$44: C72.2
- removed net N$45: C72.1
- removed net N$47: C71.2, R71.1
- removed net N$48: C71.1
- removed net N_ADC_PULL: D202.A, IC4.1
- removed net PHASE_ERROR: R51.1
- removed net PWR_3V3_GPS: C111.1, IC11.8
- removed net RESET: JP1.1, R41.2
- removed net SS: R21.1
- removed net TOSC1: IC4.3
- removed net VCC: C911.1, C931.1, C951.1, CON5.7, CON6.3, IC3.16, JP2.2, L31.2, R41.1, R71.2, R81.2
- removed net VCC_3V3_SJ2: SJ22.1
- new net AGND: R021.1, U1.G7, U1.H7, U1.J7
- new net FPGA_ADC_VP_0: U1.H8
- new net FPGA_DXN_0: R105.1, U1.K7
- new net FPGA_DXP_0: R104.1, U1.K8
- new net FPGA_VCCADC_0: C091.1, C092.1, R091.1, U1.G8
- new net FPGA_VCCAUX: C1021.1, C1022.1, C1023.1, C1024.1, C1025.1, C1026.1, R103.1, U1.G10, U1.J10, U1.K11, U1.L10
- new net FPGA_VCCBATT: R041.1, U1.F8
- new net FPGA_VCCBRAM: C1011.1, C1012.1, R102.1, U1.E10, U1.F11
- new net FPGA_VCCINT: C1001.1, C1002.1, C1003.1, C1004.1, C1005.1, C1006.1, R101.1, U1.F7, U1.F9, U1.G6, U1.H9, U1.J6, U1.K9, U1.L8
- new net FPGA_VCCO_0: C041.1, R042.1, U1.E7, U1.L6
- new net FPGA_VCCO_14: C051.1, C052.1, C053.1, C054.1, C055.1, C056.1, C057.1, R051.1, U1.L16, U1.M13, U1.N10, U1.P7, U1.R14, U1.T11
- new net FPGA_VCCO_15: C062.1, C063.1, C064.1, C065.1, C066.1, C067.1, R061.1, U1.A16, U1.B13, U1.C10, U1.E14, U1.H15, U1.J12
- new net FPGA_VCCO_34: C071.1, C072.1, C073.1, R071.1, U1.M3, U1.R4, U1.T1
- new net FPGA_VCCO_35: C082.1, C083.1, C084.1, C085.1, C086.1, C087.1, R081.1, U1.A6, U1.B3, U1.D7, U1.E4, U1.F1, U1.J2
- new net GPS_2ND_RX: R152.1, U151.6
- new net GPS_2ND_TX: U151.5
- new net GPS_3DFIX: U151.13
- new net GPS_ANT: CON181.1, U151.1
- new net GPS_NRESET: R151.1, U151.7
- new net PWR_1V0: R101.2, R102.2
- new net PWR_1V25_PREC: U1.J8
- new net PWR_1V8: R041.2, R091.2, R103.2
- new net PWR_3V3: C152.1, D151.1, R031.1, R042.2, R051.2, R061.2, R071.2, R081.2, R151.2, R152.2, RP151.2, U151.16
- new net PWR_5V0: CON151.3
- new net PWR_VCTCXO_3V0: C031.1, D031.C, R031.2, U031.4
- new net REFC_20MHZ: U031.3
- new net VCTCXO_VC: U031.1
- net GND: now also C031.2, C041.2, C051.2, C052.2, C053.2, C054.2, C055.2, C056.2, C057.2, C062.2, C063.2, C064.2, C065.2, C066.2, C067.2, C071.2, C072.2, C073.2, C082.2, C083.2, C084.2, C085.2, C086.2, C087.2, C091.2, C092.2, C1001.2, C1002.2, C1003.2, C1004.2, C1005.2, C1006.2, C1011.2, C1012.2, C1021.2, C1022.2, C1023.2, C1024.2, C1025.2, C1026.2, C141.-, C142.2, C151.-, C152.2, CON141.4, CON151.1, CON151.10, CON151.9, CON181.2, CON181.3, CON181.4, CON181.5, CON182.2, CON182.3, CON183.2, CON183.3, CON183.4, CON183.5, CON184.2, CON184.3, CON184.4, CON184.5, CON185.2, CON185.3, CON185.4, CON185.5, CON186.2, CON186.3, CON186.4, CON186.5, D031.A, D141.A, D142.A, H191.B2,8, H192.B2,8, H193.B2,8, H194.B2,8, R021.2, R104.2, R105.2, R143.1, U031.2, U1.A1, U1.A11, U1.B8, U1.C15, U1.C5, U1.D12, U1.D2, U1.E9, U1.F10, U1.F16, U1.F6, U1.G13, U1.G3, U1.G9, U1.H6, U1.J11, U1.J9, U1.K14, U1.K4, U1.K6, U1.L1, U1.L11, U1.M8, U1.N15, U1.N5, U1.P12, U1.P2, U1.R9, U1.T16, U1.T6, U151.10, U151.15, U151.2, U151.4, U151.8; no longer C111.2, C221.2, C3.-, C31.1, C32.2, C4.2, C51.2, C81.-, C911.2, C921.2, C922.2, C931.2, C951.2, CON1.2, CON1.3, CON10.2, CON10.3, CON10.4, CON10.5, CON2.4, CON3.2, CON3.3, CON3.4, CON3.5, CON4.6, CON5.10, CON5.2, CON6.1, CON6.6, CON7.2, CON7.3, CON7.4, CON7.5, CON8.2, CON8.3, CON8.4, CON8.5, CON9.2, CON9.3, CON9.4, CON9.5, D221.A, D3.A, D4.A, IC11.1, IC11.10, IC11.12, IC3.8, IC4.2, JP3.1, R52.1, R8.1, SJ21.1
- net GPS_ANT_PWR: now also CON151.4, RP151.1, U151.3; no longer RPOLY2.1
- net GPS_NMEA_RX: now also CON151.5, U151.12; no longer IC11.3
- net GPS_NMEA_TX: now also CON151.6, U151.11; no longer IC11.2, R25.1
- net GPS_PPS: now also CON151.7, U151.9; no longer IC11.4
- net PWR_BACKUP_GPS: now also C151.+, CON151.2, D151.3, U151.14; no longer C81.+, D82.3, IC11.6
- net REFC_10MHZ: now also CON182.1; no longer CON1.1
- net SIG_CH0_I: now also CON183.1; no longer CON3.1
- net SIG_CH0_Q: now also CON184.1; no longer CON8.1
- net SIG_CH1_I: now also CON185.1; no longer CON9.1
- net SIG_CH1_Q: now also CON186.1; no longer CON10.1
- net USB_5V: now also C141.+, C142.1, RP141.2; no longer C3.+, C4.1, RPOLY3.2
- net USB_DISC: now also R144.2; no longer R7.2
- net USB_D_MIN1: now also CON141.2, D142.C, R142.1, R144.1; no longer CON2.2, D3.C, R5.1, R7.1
- net USB_D_MNS: now also R142.2; no longer R5.2
- net USB_D_PLS: now also R141.2; no longer R6.2
- net USB_D_PLS1: now also CON141.3, D141.C, R141.1, R143.2; no longer CON2.3, D4.C, R6.1, R8.2
- net USB_PWR1: now also CON141.1, RP141.1; no longer CON2.1, RPOLY3.1
Routing:
- net VCC: track 289.4 -> 0.00 mm, vias 11 -> 0
- net GND: track 465.1 -> 733.7 mm, vias 22 -> 6
- net PWR_3V3: track 0.00 -> 212.2 mm, vias 0 -> 3
- net JTAG_SRST: track 147.9 -> 0.00 mm, vias 5 -> 0
- net +3V3: track 125.8 -> 0.00 mm, vias 7 -> 0
- net JTAG_TDI: track 96.8 -> 0.00 mm, vias 1 -> 0
- net GND_SJ1: track 88.7 -> 0.00 mm, vias 4 -> 0
- net ADC_PHASE: track 87.5 -> 0.00 mm, vias 3 -> 0
- net USB_DISC: track 80.8 -> 0.00 mm, vias 3 -> 0
- net FPGA_VCCINT: track 0.00 -> 73.0 mm, vias 0 -> 2
- net VCC_3V3_SJ2: track 72.9 -> 0.00 mm, vias 6 -> 0
- net FPGA_VCCAUX: track 0.00 -> 67.7 mm, vias 0 -> 2
- net N_ADC_PULL: track 66.5 -> 0.00 mm, vias 3 -> 0
- net GPS_NMEA_TX: track 78.6 -> 16.8 mm, vias 2 -> 0
- net FPGA_VCCO_14: track 0.00 -> 60.1 mm, vias 0 -> 3
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- removed copper zone on layer 16, net GND
- removed copper zone on layer 16, net GND1
- removed copper zone on layer 16, net GND2
- removed copper zone on layer 16, net GND3
Other:
- board size 214.5 x 647.9 mm -> 98.9 x 99.2 mm
- board text added: "DF4IAH 10 MHz Ref.-Osc. V 3.0"
- board text added: "Ethernet"
- board text added: "GPS-Ant. MCX"
- board text added: "SERVICE-GPS"
- board text removed: "BL"
- board text removed: "DF4IAH 10 MHz Ref.-Osc. V 2.0"
- board text removed: "DW"
- board text removed: "GPS"
- board text removed: "SPI"
- board text removed: "VT"
