File: Doc/V3.x/RefOsc10MHz_3V0.sch (EAGLE design)
At the start: 57 parts, among them CON1 SD-73100-0105, CON10 MCX-J-P-X-RA-SM1, CON2 TYCO-AMP_USBUSB-B_SMT, CON3 MCX-J-P-X-RA-SM1, CON4 AVR-ISP-6SMD, CON5 AVR-JTAG-10SMD, CON6 HEADER-2X3SMD, CON7 MCX-J-P-X-RA-SM1, CON8 MCX-J-P-X-RA-SM1, CON9 MCX-J-P-X-RA-SM1, IC11 712-RXM-GNSS-TM-B, IC3 74HCT221D, IC4 CFPT-141

Commit message: avr_DF4IAH_Bootloader - Doc - Eagle: V3.0 - update of current dev. state
Parts:
- removed C111: 100n, df4iah:C-EUC0805
- removed C221, C31, C4: 100n, rcl:C-EUC0805
- removed C3: 47uF, rcl:CPOL-EUC
- removed C32: 100p, rcl:C-EUC0805
- removed C51, C911, C921, C922, C931, C951: 10n, rcl:C-EUC0805
- removed C71: 10p, rcl:C-EUC0805
- removed C72: 33p, rcl:C-EUC0805
- removed C81: 0.22F, rcl:CPOL-EUC
- removed CON1: SD-73100-0105, df4iah:MOLEX_BNC-JACK-50R_SD-73100-0105
- removed CON10, CON3, CON7, CON8, CON9: MCX-J-P-X-RA-SM1, df4iah:MCX-J-P-X-RA-SM1
- removed CON2: TYCO-AMP_USBUSB-B_SMT, df4iah:TYCO-AMP_USBUSB-B_SMT
- removed CON4: AVR-ISP-6SMD, atmel-1:AVR-ISP-6SMD
- removed CON5: AVR-JTAG-10SMD, df4iah:AVR-JTAG-10SMD
- removed CON6: HEADER-2X3SMD, df4iah:HEADER-2X3SMD
- removed D202: BZX84-C2V7, diode:BZX84CSMD
- removed D221: BZX84-C3V0, diode:BZX84CSMD
- removed D3, D4: BZX84-C3V6, diode:BZX84CSMD
- removed D82: CRS08, diode:ZENER-DIODESOT23
- removed IC11: 712-RXM-GNSS-TM-B, df4iah:712-RXM-GNSS-TM-B
- removed IC3: 74HCT221D, 74xx-eu:74HCT221D
- removed IC4: CFPT-141, df4iah:CFPT-141
- removed JP1, JP2, JP3: (no value), jumper:SJW
- removed L31: 10uH, rcl:L-EUL1812
- removed LFP111: WE-CBF_300R, df4iah:L-EUL3216C
- removed R21, R22, R23, R25: 2.7k, rcl:R-EU_R0805
- removed R221: 56, rcl:R-EU_R0805
- removed R41: 12k, rcl:R-EU_R0805
- removed R5, R6: 68, rcl:R-EU_R0805
- removed R51, R52, R81: 1k, rcl:R-EU_R0805
- removed R7, R71: 1.5k, rcl:R-EU_R0805
- removed R8: 1M, rcl:R-EU_R0805
- removed RPOLY2: 1206L012WR_0.1A, rcl:R-EU_M1206
- removed RPOLY3: 1206L025YR_0.5A, rcl:R-EU_M1206
- removed SJ21, SJ22: (no value), jumper:SJ
- added C031, C142: 100n, rcl:C-EUC0805
- added C041, C1011, C1021: 47uF, rcl:C-EUC0805
- added C051, C1001: 100uF, rcl:C-EUC1206
- added C052, C053, C062, C063, C071, C082, C083, C091, C1002, C1003, C1022, C1023: 4.7uF, rcl:C-EUC0402
- added C054, C055, C056, C057, C064, C065, C066, C067, C072, C073, C084, C085, C086, C087, C092, C1004, C1005, C1006, C1012, C1024, C1025, C1026: 0.47uF, rcl:C-EUC0402
- added C141: 47uF, rcl:CPOL-EUC
- added C151: 0.22F, rcl:CPOL-EUC
- added C152: 100n, df4iah:C-EUC0805
- added CON141: TYCO-AMP_USBUSB-B_SMT, df4iah:TYCO-AMP_USBUSB-B_SMT
- added CON151: HEADER-2X5SMD, df4iah_connector:HEADER-2X5SMD
- added CON181, CON183, CON184, CON185, CON186: MCX-J-P-X-RA-SM1, df4iah:MCX-J-P-X-RA-SM1
- added CON182: SD-73100-0105, df4iah:MOLEX_BNC-JACK-50R_SD-73100-0105
- added CON191: HEADER-2X3SMD, df4iah:HEADER-2X3SMD
- added CON192: AVR-JTAG-10SMD, df4iah:AVR-JTAG-10SMD
- added D031: BZX84-C3V0, diode:BZX84CSMD
- added D141, D142: BZX84-C3V6, diode:BZX84CSMD
- added D151: CRS08, diode:ZENER-DIODESOT23
- added D191: BZX84-C2V7, diode:BZX84CSMD
- added H191, H192, H193, H194: MOUNT-PAD-ROUND2.8, holes:MOUNT-PAD-ROUND2.8
- added L191: 10uH, rcl:L-EUL1812
- added R021: 0, rcl:R-EU_R0805
- added R031: 56, rcl:R-EU_R0805
- added R041, R042, R051, R061, R071, R081, R091, R101, R102, R103, R104, R105: 0, rcl:R-EU_R0402
- added R141, R142: 68, rcl:R-EU_R0805
- added R143: 1M, rcl:R-EU_R0805
- added R144: 1.5k, rcl:R-EU_R0805
- added R151, R152: 10k, rcl:R-EU_R0805
- added RP141: 1206L025YR_0.5A, rcl:R-EU_M1206
- added RP151: 1206L012WR_0.1A, rcl:R-EU_M1206
- added U031: CFPT-141, df4iah:CFPT-141
- added U1: XC7A35TFTG256, df4iah_fpga:XC7A35TFTG256
- added U151: GLOBALTOP-FIREFLY1-GMM-G3, df4iah_gps:GLOBALTOP-FIREFLY1-GMM-G3
Connections:
- removed net +3V0: C221.1, D221.C, IC4.VCC_3V0, R221.2
- removed net +3V3: C921.1, C922.1, CON6.5, D202.C, D82.A, R221.1, RPOLY2.2, SJ22.2
- removed net 14: IC11.14, LFP111.1
- removed net ADC_PHASE: R52.2
- removed net ADC_PHASE_PULLHOLD: C51.1, R51.2
- removed net AREF: C32.1
- removed net AVCC: C31.2, L31.1
- removed net CPLD_GPS_NMEA_TX: R25.2
- removed net GND_SJ1: SJ21.2
- removed net GPS_HF: CON7.1, IC11.11, LFP111.2
- removed net INT1: JP3.2
- removed net ISP_MISO: CON4.1, R22.1
- removed net ISP_MOSI: CON4.4
- removed net ISP_SCK: CON4.3, R23.2
- removed net ISP_VTARGET: CON4.2, JP2.1
- removed net JTAG_SRST: CON4.5, CON5.6, JP1.2, R21.2
- removed net JTAG_TCK: CON5.1
- removed net JTAG_TDI: CON5.9
- removed net JTAG_TDO: CON5.3
- removed net JTAG_TMS: CON5.5
- removed net JTAG_VREF: CON5.4, R81.1
- removed net MISO: R22.2
- removed net N$1: CON6.2
- removed net N$3: CON6.4
- removed net N$44: C72.2
- removed net N$45: C72.1
- removed net N$47: C71.2, R71.1
- removed net N$48: C71.1
- removed net N_ADC_PULL: D202.A, IC4.VC
- removed net PHASE_ERROR: R51.1
- removed net PWR_3V3_GPS: C111.1, IC11.8
- removed net RESET: JP1.1, R41.2
- removed net SS: R21.1
- removed net TOSC1: IC4.OUT
- removed net VCC: C911.1, C931.1, C951.1, CON5.7, CON6.3, IC3P.VCC, JP2.2, L31.2, R41.1, R71.2, R81.2
- removed net VCC_3V3_SJ2: SJ22.1
- new net AGND: R021.1, U1BXADC.GNDADC_0, U1BXADC.VN_0, U1BXADC.VREFN_0
- new net FPGA_ADC_VP_0: U1BXADC.VP_0
- new net FPGA_DXN_0: R105.1, U1BTDIODE.DXN_0
- new net FPGA_DXP_0: R104.1, U1BTDIODE.DXP_0
- new net FPGA_VCCADC_0: C091.1, C092.1, R091.1, U1BXADC.VCCADC_0
- new net FPGA_VCCAUX: C1021.1, C1022.1, C1023.1, C1024.1, C1025.1, C1026.1, R103.1, U1BVCCAUX.VCCAUX@0, U1BVCCAUX.VCCAUX@1, U1BVCCAUX.VCCAUX@2, U1BVCCAUX.VCCAUX@3
- new net FPGA_VCCBATT: R041.1, U1B0.VCCBATT_0
- new net FPGA_VCCBRAM: C1011.1, C1012.1, R102.1, U1BVCCBRAM.VCCBRAM@0, U1BVCCBRAM.VCCBRAM@1
- new net FPGA_VCCINT: C1001.1, C1002.1, C1003.1, C1004.1, C1005.1, C1006.1, R101.1, U1BVCCINT.VCCINT@0, U1BVCCINT.VCCINT@1, U1BVCCINT.VCCINT@2, U1BVCCINT.VCCINT@3, U1BVCCINT.VCCINT@4, U1BVCCINT.VCCINT@5, U1BVCCINT.VCCINT@6
- new net FPGA_VCCO_0: C041.1, R042.1, U1B0.CFGBVS_0, U1B0.VCCO_0
- new net FPGA_VCCO_14: C051.1, C052.1, C053.1, C054.1, C055.1, C056.1, C057.1, R051.1, U1B14.VCCO_14@0, U1B14.VCCO_14@1, U1B14.VCCO_14@2, U1B14.VCCO_14@3, U1B14.VCCO_14@4, U1B14.VCCO_14@5
- new net FPGA_VCCO_15: C062.1, C063.1, C064.1, C065.1, C066.1, C067.1, R061.1, U1B15.VCCO_15@0, U1B15.VCCO_15@1, U1B15.VCCO_15@2, U1B15.VCCO_15@3, U1B15.VCCO_15@4, U1B15.VCCO_15@5
- new net FPGA_VCCO_34: C071.1, C072.1, C073.1, R071.1, U1B34.VCCO_34@0, U1B34.VCCO_34@1, U1B34.VCCO_34@2
- new net FPGA_VCCO_35: C082.1, C083.1, C084.1, C085.1, C086.1, C087.1, R081.1, U1B35.VCCO_35@0, U1B35.VCCO_35@1, U1B35.VCCO_35@2, U1B35.VCCO_35@3, U1B35.VCCO_35@4, U1B35.VCCO_35@5
- new net GPS_2ND_RX: R152.1, U151.RXDB
- new net GPS_2ND_TX: U151.TXDB
- new net GPS_3DFIX: U151.3D_FIX
- new net GPS_ANT: CON181.1, U151.ANTENNA_IN
- new net GPS_NRESET: R151.1, U151.NRESET
- new net PWR_1V0: R101.2, R102.2
- new net PWR_1V25_PREC: U1BXADC.VREFP_0
- new net PWR_1V8: R041.2, R091.2, R103.2
- new net PWR_3V3: C152.1, D151.A, R031.1, R042.2, R051.2, R061.2, R071.2, R081.2, R151.2, R152.2, RP151.2, U151.VCC_3V3
- new net PWR_5V0: CON151.3
- new net PWR_VCTCXO_3V0: C031.1, D031.C, R031.2, U031.VCC_3V0
- new net REFC_20MHZ: U031.OUT
- new net VCTCXO_VC: U031.VC
- net GND: now also C031.2, C041.2, C051.2, C052.2, C053.2, C054.2, C055.2, C056.2, C057.2, C062.2, C063.2, C064.2, C065.2, C066.2, C067.2, C071.2, C072.2, C073.2, C082.2, C083.2, C084.2, C085.2, C086.2, C087.2, C091.2, C092.2, C1001.2, C1002.2, C1003.2, C1004.2, C1005.2, C1006.2, C1011.2, C1012.2, C1021.2, C1022.2, C1023.2, C1024.2, C1025.2, C1026.2, C141.-, C142.2, C151.-, C152.2, CON141.GND, CON151.1, CON151.10, CON151.9, CON181.2, CON181.3, CON181.4, CON181.5, CON182.2, CON182.3, CON183.2, CON183.3, CON183.4, CON183.5, CON184.2, CON184.3, CON184.4, CON184.5, CON185.2, CON185.3, CON185.4, CON185.5, CON186.2, CON186.3, CON186.4, CON186.5, D031.A, D141.A, D142.A, H191.MOUNT, H192.MOUNT, H193.MOUNT, H194.MOUNT, R021.2, R104.2, R105.2, R143.1, U031.GND, U151.GND@0, U151.GND@1, U151.GND@2, U151.GND@3, U151.GND@4, U1BGND.GND@0, U1BGND.GND@1, U1BGND.GND@10, U1BGND.GND@11, U1BGND.GND@12, U1BGND.GND@13, U1BGND.GND@14, U1BGND.GND@15, U1BGND.GND@16, U1BGND.GND@17, U1BGND.GND@18, U1BGND.GND@19, U1BGND.GND@2, U1BGND.GND@20, U1BGND.GND@21, U1BGND.GND@22, U1BGND.GND@23, U1BGND.GND@24, U1BGND.GND@25, U1BGND.GND@26, U1BGND.GND@27, U1BGND.GND@28, U1BGND.GND@29, U1BGND.GND@3, U1BGND.GND@4, U1BGND.GND@5, U1BGND.GND@6, U1BGND.GND@7, U1BGND.GND@8, U1BGND.GND@9; no longer C111.2, C221.2, C3.-, C31.1, C32.2, C4.2, C51.2, C81.-, C911.2, C921.2, C922.2, C931.2, C951.2, CON1.2, CON1.3, CON10.2, CON10.3, CON10.4, CON10.5, CON2.GND, CON3.2, CON3.3, CON3.4, CON3.5, CON4.6, CON5.10, CON5.2, CON6.1, CON6.6, CON7.2, CON7.3, CON7.4, CON7.5, CON8.2, CON8.3, CON8.4, CON8.5, CON9.2, CON9.3, CON9.4, CON9.5, D221.A, D3.A, D4.A, IC11.1, IC11.10, IC11.12, IC3P.GND, IC4.GND, JP3.1, R52.1, R8.1, SJ21.1
- net GPS_ANT_PWR: now also CON151.4, RP151.1, U151.VANT; no longer RPOLY2.1
- net GPS_NMEA_RX: now also CON151.5, U151.RXDA; no longer IC11.3
- net GPS_NMEA_TX: now also CON151.6, U151.TXDA; no longer IC11.2, R25.1
- net GPS_PPS: now also CON151.7, U151.1PPS; no longer IC11.4
- net PWR_BACKUP_GPS: now also C151.+, CON151.2, D151.C, U151.VBACKUP; no longer C81.+, D82.C, IC11.6
- net REFC_10MHZ: now also CON182.1; no longer CON1.1
- net SIG_CH0_I: now also CON183.1; no longer CON3.1
- net SIG_CH0_Q: now also CON184.1; no longer CON8.1
- net SIG_CH1_I: now also CON185.1; no longer CON9.1
- net SIG_CH1_Q: now also CON186.1; no longer CON10.1
- net USB_5V: now also C141.+, C142.1, RP141.2; no longer C3.+, C4.1, RPOLY3.2
- net USB_DISC: now also R144.2; no longer R7.2
- net USB_D_MIN1: now also CON141.D-, D142.C, R142.1, R144.1; no longer CON2.D-, D3.C, R5.1, R7.1
- net USB_D_MNS: now also R142.2; no longer R5.2
- net USB_D_PLS: now also R141.2; no longer R6.2
- net USB_D_PLS1: now also CON141.D+, D141.C, R141.1, R143.2; no longer CON2.D+, D4.C, R6.1, R8.2
- net USB_PWR1: now also CON141.VBUS, RP141.1; no longer CON2.VBUS, RPOLY3.1
Other:
- note added: "DF4IAH 10 MHz Reference Oscillator V 3.0"
- note added: "Ethernet"
- note added: "FLASH"
- note added: "S0"
- note added: "S1"
- note added: "S2"
- note added: "S3"
- note added: "S4"
- note added: "S5"
- note added: "S6"
- note added: "S7"
- note added: "SDRAM"
- note added: "Sockets"
- note added: "XILINX Artix XC7A35TFTG256"
- note removed: "10 MHz out"
- note removed: "10 kHz"
- note removed: "2.5 MHz out"
- note removed: "20 MHz in"
- note removed: "ADC-Phase"
- note removed: "ADC-Pull"
- note removed: "AVR - PINs: - PB0 20 MHz Clock Out (ICP) - PB1 USB Disconnect (DigOut) - PB2 ISP SS (SS) - PB3 ISP MOSI (MOSI) - PB4 ISP MISO (MISO) - PB5 ISP SCK (SCK) - PB6 Crystal 20 MHz In (XTAL1) - PB7 Crystal 20 MHz Out (XTAL2) - PC0 ADC0 Pull Voltage (ADC0) - PC1 ADC1 Phase Error (ADC1) - PC2 USB D+ (DigIn/DigOut) - PC3 USB D- (DigIn/DigOut) - PC4 reserved (I2C SDA) - PC5 reserved (I2C SCL) - PD0 GPS Data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"
- note removed: "Bootloader"
- note removed: "CPLD_SER_GPS"
- note removed: "DF4IAH 10 MHz Reference Oscillator V 2.0"
- note removed: "GPS-Module"
- note removed: "Gate"
- note removed: "Gate Trig out"
- note removed: "Gate in"
- note removed: "I2C"
- note removed: "I2C - PINs: 1 GND 2 SCL 3 VCC 5V 4 SDA 5 3.3V 6 GND"
- note removed: "IC-Supplies"
- note removed: "JTAG_TCK"
- note removed: "JTAG_TDI"
- note removed: "JTAG_TDO"
- note removed: "JTAG_TMS"
- note removed: "MMU"
- note removed: "NC"
- note removed: "PPS"
- note removed: "Phase out"
- note removed: "Phase-Error"
- note removed: "Pull & Hold"
- note removed: "RESET in"
- note removed: "SPI - PINs: 1 MISO 2 V-Target 3 SCK 4 MOSI 5 RST 6 GND"
- note removed: "Sync"
- note removed: "Sync in"
- note removed: "USB D+"
- note removed: "USB D-"
- note removed: "USB Disconnect"
- note removed: "VTarget"
- note removed: "debugWIRE"
- note removed: "t=33ns"
- note removed: "t=362ns"
