File: Doc/V2.x/RefOsc10MHz_2V2.sch (EAGLE design)
At the start: 83 parts, among them CON1 TYCO-AMP_USBUSB-B_SMT, CON2 HEADER-2X5SMD, CON3 SD-73100-0105, CON4 AVR-ISP-6SMD, CON5 AVR-JTAG-10SMD, CON6 HEADER-2X3SMD, CON7 MCX-J-P-X-RA-SM1, IC1 ATmega328-P, IC2 LC4032V_XXT44, IC3 74HCT221D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

Commit message: avr_DF4IAH_Bootloader - Doc - Eagle: V2.2 - correction: CRS80 --> CRS08
Parts:
- D611, D921: value CRS80 -> CRS08
Changed lines of the file:
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@@
 <part name="GND24" library="supply1" deviceset="GND" device=""/>
 <part name="C921" library="rcl" deviceset="CPOL-EU" device="140CLH-1010" value="0.22F"/>
-<part name="D611" library="diode" deviceset="ZENER-DIODE" device="SOD80C" value="CRS80"/>
-<part name="D921" library="diode" deviceset="ZENER-DIODE" device="SOD80C" value="CRS80"/>
+<part name="D611" library="diode" deviceset="ZENER-DIODE" device="SOD80C" value="CRS08"/>
+<part name="D921" library="diode" deviceset="ZENER-DIODE" device="SOD80C" value="CRS08"/>
 <part name="D701" library="diode" deviceset="BZX84CSMD" device="" value="BZX84-C3V0"/>
 <part name="R701" library="rcl" deviceset="R-EU_" device="R0805" value="68"/>

Commit message: avr_DF4IAH_Bootloader - Doc - Eagle: V2.2 - correction: MCX socket ground not completed
Other:
- note added: "DF4IAH 10 MHz Reference Oscillator V 2.2a with GlobalTop FireFly 1 (includes MediaTek MT3333)"
- note removed: "DF4IAH 10 MHz Reference Oscillator V 2.2 with GlobalTop FireFly 1 (includes MediaTek MT3333)"
Changed lines of the file:
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@@
 <text x="193.04" y="147.574" size="1.016" layer="97">2.5 MHz out</text>
 <text x="0.254" y="294.386" size="2.54" layer="97">DF4IAH  10 MHz Reference Oscillator
-V 2.2
+V 2.2a
 with GlobalTop FireFly 1 (includes MediaTek MT3333)</text>
 <text x="54.356" y="146.558" size="1.778" layer="97">USB Disconnect</text>

Commit message: avr_DF4IAH_Bootloader - Doc - Eagle: V2.1/V2.2 - removed elkos and replaced it by C0805 MLCCs
Parts:
- C151, C211, C612, C613: device rcl:CPOL-EUB -> rcl:C-EUC0805
- C911: device rcl:CPOL-EUC -> rcl:C-EUC0805
Connections:
- net +3V3: now also C612.1, C613.1; no longer C612.+, C613.+
- net GND: now also C151.2, C211.2, C612.2, C613.2, C911.2; no longer C151.-, C211.-, C612.-, C613.-, C911.-
- net N_ADC_PULL: now also C151.1; no longer C151.+
- net VCC: now also C211.1, C911.1; no longer C211.+, C911.+
Changed lines of the file:
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@@
 <part name="P+12" library="supply1" deviceset="VCC" device=""/>
 <part name="GND16" library="supply1" deviceset="GND" device=""/>
-<part name="C911" library="rcl" deviceset="CPOL-EU" device="C" value="47uF"/>
+<part name="C911" library="rcl" deviceset="C-EU" device="C0805" value="47uF"/>
 <part name="D911" library="diode" deviceset="BZX84CSMD" device="" value="BZX84-C3V6"/>
 <part name="D912" library="diode" deviceset="BZX84CSMD" device="" value="BZX84-C3V6"/>
@@
 <part name="C391" library="rcl" deviceset="C-EU" device="C0805" value="100n"/>
 <part name="C591" library="rcl" deviceset="C-EU" device="C0805" value="10n"/>
-<part name="C151" library="rcl" deviceset="CPOL-EU" device="B" value="10uF"/>
+<part name="C151" library="rcl" deviceset="C-EU" device="C0805" value="10uF"/>
 <part name="R612" library="rcl" deviceset="R-EU_" device="R0805" value="45.3k"/>
 <part name="R611" library="rcl" deviceset="R-EU_" device="R0805" value="10k"/>
@@
 <part name="R132" library="rcl" deviceset="R-EU_" device="R0805" value="47k"/>
 <part name="R311" library="rcl" deviceset="R-EU_" device="R0805" value="4.7k"/>
-<part name="C612" library="rcl" deviceset="CPOL-EU" device="B" value="22uF"/>
-<part name="C613" library="rcl" deviceset="CPOL-EU" device="B" value="22uF"/>
-<part name="C211" library="rcl" deviceset="CPOL-EU" device="B" value="22uF"/>
+<part name="C612" library="rcl" deviceset="C-EU" device="C0805" value="22uF"/>
+<part name="C613" library="rcl" deviceset="C-EU" device="C0805" value="22uF"/>
+<part name="C211" library="rcl" deviceset="C-EU" device="C0805" value="22uF"/>
 <part name="U8" library="df4iah_gps" deviceset="GLOBALTOP-FIREFLY1-GMM-G3" device=""/>
 <part name="GND25" library="df4iah" deviceset="GND" device=""/>
@@
 <pinref part="D151" gate="G$1" pin="A"/>
 <pinref part="C152" gate="G$1" pin="2"/>
-<pinref part="C151" gate="G$1" pin="-"/>
+<pinref part="C151" gate="G$1" pin="2"/>
 <junction x="25.4" y="167.64"/>
 </segment>
@@
 <pinref part="IC7" gate="&gt;NAME" pin="GND"/>
 <pinref part="D611" gate="G$1" pin="A"/>
-<pinref part="C612" gate="G$1" pin="-"/>
-<pinref part="C613" gate="G$1" pin="-"/>
-<pinref part="C211" gate="G$1" pin="-"/>
+<pinref part="C612" gate="G$1" pin="2"/>
+<pinref part="C613" gate="G$1" pin="2"/>
+<pinref part="C211" gate="G$1" pin="2"/>
 </segment>
 <segment>
@@
 <pinref part="GND1" gate="1" pin="GND"/>
 <wire x1="17.78" y1="101.6" x2="17.78" y2="106.68" width="0.1524" layer="91"/>
-<pinref part="C911" gate="G$1" pin="-"/>
+<pinref part="C911" gate="G$1" pin="2"/>
 <pinref part="D911" gate="G$1" pin="A"/>
 <pinref part="D912" gate="G$1" pin="A"/>
@@
 <pinref part="L101" gate="G$1" pin="2"/>
 <pinref part="IC6" gate="A" pin="VIN"/>
-<pinref part="C211" gate="G$1" pin="+"/>
+<pinref part="C211" gate="G$1" pin="1"/>
 </segment>
 <segment>
@@
 <wire x1="20.32" y1="149.86" x2="20.32" y2="144.78" width="0.1524" layer="91"/>
 <junction x="20.32" y="144.78"/>
-<pinref part="C911" gate="G$1" pin="+"/>
+<pinref part="C911" gate="G$1" pin="1"/>
 <pinref part="RPOLY1" gate="G$1" pin="2"/>
 <pinref part="C912" gate="G$1" pin="1"/>
@@
 <junction x="25.4" y="177.8"/>
 <pinref part="R151" gate="G$1" pin="2"/>
-<pinref part="C151" gate="G$1" pin="+"/>
+<pinref part="C151" gate="G$1" pin="1"/>
 <pinref part="IC7" gate="&gt;NAME" pin="VC"/>
 <pinref part="D152" gate="G$1" pin="A"/>
@@
 <junction x="116.84" y="266.7"/>
 <pinref part="R701" gate="G$1" pin="1"/>
-<pinref part="C612" gate="G$1" pin="+"/>
-<pinref part="C613" gate="G$1" pin="+"/>
-</segment>
-</net>
+<pinref part="C612" gate="G$1" pin="1"/>
+<pinref part="C613" gate="G$1" pin="1"/>
+</segment>
+</net>

Commit message: avr_DF4IAH_Bootloader - Doc - Eagle: 2.1, 2.2, 2.3 - three resistors changed
Parts:
- R311: value 4.7k -> 4.3k
- R611: value 10k -> 15k
- R612: value 45.3k -> 68k
Changed lines of the file:
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@@
 <part name="C591" library="rcl" deviceset="C-EU" device="C0805" value="10n"/>
 <part name="C151" library="rcl" deviceset="C-EU" device="C0805" value="10uF"/>
-<part name="R612" library="rcl" deviceset="R-EU_" device="R0805" value="45.3k"/>
-<part name="R611" library="rcl" deviceset="R-EU_" device="R0805" value="10k"/>
+<part name="R612" library="rcl" deviceset="R-EU_" device="R0805" value="68k"/>
+<part name="R611" library="rcl" deviceset="R-EU_" device="R0805" value="15k"/>
 <part name="R601" library="rcl" deviceset="R-EU_" device="R0805" value="100k"/>
 <part name="L611" library="rcl" deviceset="L-EU" device="L5650M" value="4.7uH"/>
@@
 <part name="R131" library="rcl" deviceset="R-EU_" device="R0805" value="15k"/>
 <part name="R132" library="rcl" deviceset="R-EU_" device="R0805" value="47k"/>
-<part name="R311" library="rcl" deviceset="R-EU_" device="R0805" value="4.7k"/>
+<part name="R311" library="rcl" deviceset="R-EU_" device="R0805" value="4.3k"/>
 <part name="C612" library="rcl" deviceset="C-EU" device="C0805" value="22uF"/>
 <part name="C613" library="rcl" deviceset="C-EU" device="C0805" value="22uF"/>
