File: Doc/V2.x/RefOsc10MHz_2V3.sch (EAGLE design)
At the start: 82 parts, among them CON1 TYCO-AMP_USBUSB-B_SMT, CON2 HEADER-2X5SMD, CON3 SD-73100-0105, CON4 AVR-ISP-6SMD, CON5 AVR-JTAG-10SMD, CON6 HEADER-2X3SMD, CON7 MCX-J-P-X-RA-SM1, U1 ATmega328-P, U2 LC4032V_XXT44, U3 74HCT221D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

Commit message: avr_DF4IAH_Bootloader - Doc - Eagle: 2.1, 2.2, 2.3 - three resistors changed
Parts:
- R311: value 4.7k -> 4.3k
- R611: value 10k -> 15k
- R612: value 45.3k -> 68k
Changed lines of the file:
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@@
 <part name="C591" library="rcl" deviceset="C-EU" device="C0805" value="10n"/>
 <part name="C151" library="rcl" deviceset="C-EU" device="C0805" value="10uF"/>
-<part name="R612" library="rcl" deviceset="R-EU_" device="R0805" value="45.3k"/>
-<part name="R611" library="rcl" deviceset="R-EU_" device="R0805" value="10k"/>
+<part name="R612" library="rcl" deviceset="R-EU_" device="R0805" value="68k"/>
+<part name="R611" library="rcl" deviceset="R-EU_" device="R0805" value="15k"/>
 <part name="R601" library="rcl" deviceset="R-EU_" device="R0805" value="100k"/>
 <part name="L611" library="rcl" deviceset="L-EU" device="L5650M" value="4.7uH"/>
@@
 <part name="R131" library="rcl" deviceset="R-EU_" device="R0805" value="15k"/>
 <part name="R132" library="rcl" deviceset="R-EU_" device="R0805" value="47k"/>
-<part name="R311" library="rcl" deviceset="R-EU_" device="R0805" value="4.7k"/>
+<part name="R311" library="rcl" deviceset="R-EU_" device="R0805" value="4.3k"/>
 <part name="C612" library="rcl" deviceset="C-EU" device="C0805" value="22uF"/>
 <part name="C613" library="rcl" deviceset="C-EU" device="C0805" value="22uF"/>
