File: Doc/V2.x/RefOsc10MHz_2V3.sch (EAGLE design)
At the start: 72 parts, among them CON1 TYCO-AMP_USBUSB-B_SMT, CON2 HEADER-2X5, CON3 SD-73100-0105, CON5 AVR-JTAG-10, CON6 HEADER-2X3, CON7 MCX-J-P-X-RA-SM1, U1 ATmega328-P, U2 LC4032V_XXT44, U3 74HCT221D, U5 OPA354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

Commit message: Doc - V2.3e - via 0.6mm --> 0.35mm
Other:
- note added: "DF4IAH 10 MHz Reference Oscillator V 2.3e"
- note removed: "DF4IAH 10 MHz Reference Oscillator V 2.3d"
Changed lines of the file:
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@@
 <text x="198.12" y="145.034" size="1.016" layer="97">2.5 MHz out</text>
 <text x="5.334" y="291.846" size="2.54" layer="97">DF4IAH  10 MHz Reference Oscillator
-V 2.3d</text>
+V 2.3e</text>
 <text x="59.436" y="144.018" size="1.778" layer="97">USB Disconnect</text>
 <text x="102.616" y="122.936" size="1.778" layer="97">USB D-</text>
