File: Doc/V2.x/10MHzRefOsc_2V1.brd (EAGLE design)
At the start: 90 x 70 mm, 82 parts, among them CON1 TYCO-AMP_USBUSB-B_SMT, CON2 HEADER-2X5SMD, CON3 SD-73100-0105, CON4 AVR-ISP-6SMD, CON5 AVR-JTAG-10SMD, CON6 HEADER-2X3SMD, CON7 MCX-J-P-X-RA-SM1, IC1 ATmega328-P, IC2 LC4032V_XXT44, IC3 74HCT221D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

Commit message: avr_DF4IAH_Bootloader - Doc - Eagle: 2.1 - 3.3V adjusting resistors corrected, 2-way jumpers now THT instead of SMT
Parts:
- JP111, JP121, JP941: device jumper:SJW -> jumper:JP1
- R132: value 47k -> 51k
- turned JP111 to 180 degrees
- turned JP121 to 180 degrees
- turned JP941 to 180 degrees
Connections:
- net GND: now also JP121.2; no longer JP121.1
- net INT1: now also JP121.1; no longer JP121.2
- net ISP_VTARGET: now also JP941.2; no longer JP941.1
- net VCC: now also JP941.1; no longer JP941.2
Routing:
- net JTAG_SRST: track 162.4 -> 163.8 mm
Other:
- board text added: "DF4IAH 10 MHz Ref.-Osc. V 2.1b"
- board text removed: "DF4IAH 10 MHz Ref.-Osc. V 2.1a"
