File: Doc/V2.x/10MHzRefOsc_2V2.brd (EAGLE design)
At the start: 90 x 70 mm, 83 parts, among them CON1 TYCO-AMP_USBUSB-B_SMT, CON2 HEADER-2X5SMD, CON3 SD-73100-0105, CON4 AVR-ISP-6SMD, CON5 AVR-JTAG-10SMD, CON6 HEADER-2X3SMD, CON7 MCX-J-P-X-RA-SM1, IC1 ATmega328-P, IC2 LC4032V_XXT44, IC3 74HCT221D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

Commit message: avr_DF4IAH_Bootloader - Doc - Eagle: 2.2 - 3.3V adjusting resistors corrected
Parts:
- R132: value 47k -> 51k
Changed lines of the file:
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@@
 <attribute name="VALUE" x="35.93920625" y="43.547821875" size="1.016" layer="27" rot="R90"/>
 </element>
-<element name="R132" library="rcl" package="R0805" value="47k" x="33.02" y="41.91" smashed="yes" rot="R270">
+<element name="R132" library="rcl" package="R0805" value="51k" x="33.02" y="41.91" smashed="yes" rot="R270">
 <attribute name="NAME" x="33.308890625" y="37.01970625" size="1.016" layer="25" rot="R90"/>
 <attribute name="VALUE" x="33.287240625" y="43.547825" size="1.016" layer="27" rot="R90"/>
