File: Doc/V2.x/10MHzRefOsc_2V2.sch (EAGLE design)
At the start: 83 parts, among them CON1 TYCO-AMP_USBUSB-B_SMT, CON2 HEADER-2X5SMD, CON3 SD-73100-0105, CON4 AVR-ISP-6SMD, CON5 AVR-JTAG-10SMD, CON6 HEADER-2X3SMD, CON7 MCX-J-P-X-RA-SM1, IC1 ATmega328-P, IC2 LC4032V_XXT44, IC3 74HCT221D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

Commit message: avr_DF4IAH_Bootloader - Doc - Eagle: 2.2 - 3.3V adjusting resistors corrected
Parts:
- R132: value 47k -> 51k
Changed lines of the file:
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@@
 <part name="R201" library="rcl" deviceset="R-EU_" device="R0805" value="2.7k"/>
 <part name="R131" library="rcl" deviceset="R-EU_" device="R0805" value="15k"/>
-<part name="R132" library="rcl" deviceset="R-EU_" device="R0805" value="47k"/>
+<part name="R132" library="rcl" deviceset="R-EU_" device="R0805" value="51k"/>
 <part name="R311" library="rcl" deviceset="R-EU_" device="R0805" value="4.3k"/>
 <part name="C612" library="rcl" deviceset="C-EU" device="C0805" value="22uF"/>
