File: Doc/V2.x/10MHzRefOsc_2V3.sch (EAGLE design)
At the start: 82 parts, among them CON1 TYCO-AMP_USBUSB-B_SMT, CON2 HEADER-2X5SMD, CON3 SD-73100-0105, CON4 AVR-ISP-6SMD, CON5 AVR-JTAG-10SMD, CON6 HEADER-2X3SMD, CON7 MCX-J-P-X-RA-SM1, U1 ATmega328-P, U2 LC4032V_XXT44, U3 74HCT221D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

Commit message: avr_DF4IAH_Bootloader - Doc - Eagle: 2.3 - 3.3V adjusting resistors corrected, 2-way jumpers now THT instead of SMT, GPS-chip package enhanced
Parts:
- JP111, JP121, JP941: device jumper:SJW -> jumper:JP1E
- R132: value 47k -> 51k
Connections:
- net GND: now also JP121.2; no longer JP121.1
- net INT1: now also JP121.1; no longer JP121.2
- net ISP_VTARGET: now also JP941.2; no longer JP941.1
- net VCC: now also JP941.1; no longer JP941.2
Other:
- note added: "DF4IAH 10 MHz Reference Oscillator V 2.1b"
- note removed: "DF4IAH 10 MHz Reference Oscillator V 2.1a"
