File: Doc/V2.x/RefOsc10MHz_2V3.brd (EAGLE design)
At the start: 90 x 70 mm, 72 parts, among them CON1 TYCO-AMP_USBUSB-B_SMT, CON2 HEADER-2X5, CON3 SD-73100-0105, CON5 AVR-JTAG-10, CON6 HEADER-2X3, CON7 MCX-J-P-X-RA-SM1, U1 ATmega328-P, U2 LC4032V_XXT44, U3 74HCT221D, U5 OPA354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

Commit message: Doc - V2.3e - via 0.6mm --> 0.35mm
Other:
- board text added: "DF4IAH 10 MHz Ref.-Osc. V 2.3e"
- board text removed: "DF4IAH 10 MHz Ref.-Osc. V 2.3d"
Changed lines of the file:
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@@
 <text x="75.940734375" y="65.306415625" size="1.27" layer="26" font="vector" ratio="18" distance="61" rot="MR0" align="center-left">DF4IAH
 10 MHz Ref.-Osc.
-V 2.3d</text>
+V 2.3e</text>
 <text x="6.35" y="10.16" size="1.27" layer="16" font="vector" ratio="20" distance="40" rot="MR0">Bot</text>
 <text x="2.54" y="10.16" size="1.27" layer="1" font="vector" ratio="20" distance="40">Top</text>
@@
 <via x="54" y="36.625" extent="1-16" drill="0.35"/>
 <via x="13.875" y="23.625" extent="1-16" drill="0.35"/>
-<via x="26.7599625" y="44.339309375" extent="1-16" drill="0.6"/>
+<via x="26.7599625" y="44.339309375" extent="1-16" drill="0.35"/>
 <wire x1="27.82" y1="42.54" x2="29.21" y2="42.54" width="0.508" layer="1"/>
 <wire x1="26.7599625" y1="44.339309375" x2="27.82" y2="42.54" width="0.508" layer="1"/>
